File: kit-semaforo.kicad_pcb (KiCad board)
At the start: 2 copper layers, 16 x 80 mm, 12 parts, among them P1 CONN_02X04

Commit message: v0.1a enviado a fabricación
Routing:
- net GNDREF: track 63.6 -> 64.3 mm
Other:
- board text added: "v0.1a"
Changed lines of the file:
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@@
     (area 142.5 62.5 178.85 162.500001)
     (thickness 1.6)
-    (drawings 36)
-    (tracks 89)
+    (drawings 37)
+    (tracks 90)
     (zones 0)
     (modules 12)
@@
       (net 10 /PEATONES-VERDE))
   )
+  (gr_text v0.1a (at 163 125 90) (layer B.SilkS)
+    (effects (font (size 1 1) (thickness 0.2)) (justify mirror))
+  )
   (gr_text fabricadigital.org (at 166.75 91.25 90) (layer F.SilkS)
     (effects (font (size 1 1) (thickness 0.25)))
@@
   (gr_line (start 152 80) (end 152 102) (layer Edge.Cuts) (width 0.15))
   (gr_arc (start 160 80) (end 152 80) (angle 180) (layer Edge.Cuts) (width 0.15))
+  (segment (start 161.27 149.81) (end 162.472081 149.81) (width 0.25) (layer B.Cu) (net 1))
+  (segment (start 162.472081 149.81) (end 163 149.282081) (width 0.25) (layer B.Cu) (net 1))
+  (segment (start 163 149.282081) (end 163 139) (width 0.25) (layer B.Cu) (net 1))
+  (segment (start 163 139) (end 162.5 138.5) (width 0.25) (layer B.Cu) (net 1))
   (segment (start 160.75 114.75) (end 162.25 113.25) (width 0.25) (layer B.Cu) (net 1))
   (segment (start 160.25 115.25) (end 160.75 114.75) (width 0.25) (layer B.Cu) (net 1))
@@
   (segment (start 162.5 138.5) (end 158.5 138.5) (width 0.25) (layer B.Cu) (net 1))
   (via (at 158.5 138.5) (size 0.6) (drill 0.3) (layers F.Cu B.Cu) (net 1))
-  (segment (start 161.27 149.81) (end 163 148.08) (width 0.25) (layer B.Cu) (net 1))
-  (segment (start 163 148.08) (end 163 139) (width 0.25) (layer B.Cu) (net 1))
-  (segment (start 163 139) (end 162.5 138.5) (width 0.25) (layer B.Cu) (net 1))
   (via (at 162.5 138.5) (size 0.6) (drill 0.3) (layers F.Cu B.Cu) (net 1))
   (segment (start 158.73 142.19) (end 158.73 140.987919) (width 0.25) (layer F.Cu) (net 2))
